File: Controller2018/main.brd (EAGLE design)
At the start: 99 x 69 mm, 111 parts, among them Q7 MOSFET-PCHANNEL, U1 TEENSY_3.0+4, U2 DRV8301

Commit message: Updated controller values to be more realistic
Parts:
- C14, C34, C35: value .1uF -> 10nF
- R25, R5, R6: value 4.7k -> 1k
Changed lines of the file:
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@@
 <?xml version="1.0" encoding="utf-8"?>
 <!DOCTYPE eagle SYSTEM "eagle.dtd">
-<eagle version="8.4.0">
+<eagle version="9.0.1">
 <drawing>
 <settings>
@@
 <layer number="25" name="tNames" color="7" fill="1" visible="no" active="yes"/>
 <layer number="26" name="bNames" color="7" fill="1" visible="no" active="yes"/>
-<layer number="27" name="tValues" color="7" fill="1" visible="no" active="yes"/>
+<layer number="27" name="tValues" color="7" fill="1" visible="yes" active="yes"/>
 <layer number="28" name="bValues" color="7" fill="1" visible="no" active="yes"/>
 <layer number="29" name="tStop" color="7" fill="3" visible="no" active="yes"/>
@@
 <param name="dpMaxLengthDifference" value="10mm"/>
 <param name="dpGapFactor" value="2.5"/>
+<param name="checkAngle" value="0"/>
 <param name="checkFont" value="1"/>
 <param name="checkRestrict" value="1"/>
 <param name="checkStop" value="0"/>
+<param name="checkValues" value="0"/>
 <param name="useDiameter" value="13"/>
 <param name="maxErrors" value="50"/>
@@
 <attribute name="PROD_ID" value="DIO-12441" x="45.5" y="64.5" size="1.778" layer="27" rot="R180" display="off"/>
 </element>
-<element name="R5" library="SparkFun-Passives" package="0603-RES" value="4.7k" x="77.5" y="41"/>
-<element name="R6" library="SparkFun-Passives" package="0603-RES" value="4.7k" x="77.5" y="38.5"/>
-<element name="R25" library="SparkFun-Passives" package="0603-RES" value="4.7k" x="77.5" y="36"/>
+<element name="R5" library="SparkFun-Passives" package="0603-RES" value="1k" x="77.5" y="41"/>
+<element name="R6" library="SparkFun-Passives" package="0603-RES" value="1k" x="77.5" y="38.5"/>
+<element name="R25" library="SparkFun-Passives" package="0603-RES" value="1k" x="77.5" y="36"/>
 <element name="C39" library="SparkFun-Passives" package="0603-CAP" value="1uF" x="59.5" y="62" rot="R90"/>
 <element name="R26" library="SparkFun-Passives" package="0603-RES" value="100k" x="62" y="62" rot="R270"/>
@@
 <attribute name="PROD_ID" value="TRANS-08285" x="89" y="11.5" size="1.778" layer="27" display="off"/>
 </element>
-<element name="C14" library="SparkFun-Passives" package="0603-CAP" value=".1uF" x="73.5" y="41" rot="R180"/>
-<element name="C34" library="SparkFun-Passives" package="0603-CAP" value=".1uF" x="73.5" y="38.5" rot="R180"/>
-<element name="C35" library="SparkFun-Passives" package="0603-CAP" value=".1uF" x="73.5" y="36" rot="R180"/>
+<element name="C14" library="SparkFun-Passives" package="0603-CAP" value="10nF" x="73.5" y="41" rot="R180"/>
+<element name="C34" library="SparkFun-Passives" package="0603-CAP" value="10nF" x="73.5" y="38.5" rot="R180"/>
+<element name="C35" library="SparkFun-Passives" package="0603-CAP" value="10nF" x="73.5" y="36" rot="R180"/>
 <element name="U$12" library="2018" package="TSSOP-14" value="OPAMP_QUAD" x="57.5" y="42" rot="R90"/>
 <element name="R31" library="SparkFun-Resistors" package="0603-RES" value="16.2k" x="51" y="35.5"/>
