File: teensy_shields/mpu6050_ic_teensy/shield.brd (EAGLE design)
At the start: 20.3 x 41.6 mm, 7 parts

Commit message: clean up
Parts:
- added U$1: DEV, Custom_old (1):DEV
- C1, C2, C3, C4: device SparkFun-Capacitors:0603 -> SparkFun-Passives:0603-CAP
- R1: value (none) -> 10k; device eagle-ltspice:R0603 -> SparkFun-Passives:0603-RES
- TEENSY: value TEENSY_3.1-3.2_ALL_PINS -> (none)
- moved C4 70.8 mm to (10.9, 19.2), flipped to the top, turned to 0 degrees
- moved C1 64.9 mm to (12.6, 22.2), flipped to the top, turned to 270 degrees
- moved MPU6050 63.9 mm to (8.89, 22.9), flipped to the top, turned to 0 degrees
- moved TEENSY 63.5 mm to (8.89, 17.8)
- moved C3 61.1 mm to (5.33, 24.4), flipped to the top, turned to 90 degrees
- moved R1 59.0 mm to (12.6, 25.5), flipped to the top, turned to 90 degrees
- moved C2 57.3 mm to (9.27, 26.5), flipped to the top, turned to 180 degrees
Routing:
- net GND: track 24.4 -> 47.5 mm
- net INT: track 14.5 -> 24.9 mm
- net VCC: track 22.5 -> 32.2 mm
- net SDA: track 7.98 -> 5.89 mm, vias 0 -> 1
- net SCL: track 8.81 -> 7.59 mm, vias 0 -> 1
- added copper zone on layer 16, net GND
Other:
- board size 20.3 x 41.6 mm -> 18 x 35.7 mm
- board text added: "MPU6050 Teensy Shield Oct. 7, 2018 Jack Proudfoot"
- board text removed: "R1"
