File: modular_battery/battery_module.sch (EAGLE design)
At the start: 141 parts

Commit message: Added FET control for CE
Parts:
- removed RC1_1, RC1_2, RC1_3, RC1_4, RC2_1, RC2_2, RC2_3, RC2_4: (no value), SparkFun-Capacitors:CAP1206
- removed U$1: EXB-2HV, Custom_old:EXB-2HV
- added ARRAY2: EXB-2HV, Custom_old:EXB-2HV
- added Q1: MOSFET-PCHANNELSOT223, Custom_old:MOSFET-PCHANNELSOT223
- added Q2: MOSFET-NCHANNELSMD, Custom_old:MOSFET-NCHANNELSMD
- added R40, R41: 47k, SparkFun-Passives:RESISTOR0603-RES
- added U$13: CL31, Custom_old:CL31
- C10, C15, C20, C25, C30, C35, C40, C5: value (none) -> 10nF
- R14, R19, R24, R29, R34, R39, R4, R9: value TBD -> 47k
- U$11: value EXB-2HV -> CL31; device Custom_old:EXB-2HV -> Custom_old:CL31
Connections:
- removed net VDIVRC_A: RC1_1.1, U$11.P$16, U$12.1IN+
- removed net VDIVRC_B: RC1_2.1, U$11.P$15, U$12.2IN+
- removed net VDIVRC_C: RC1_3.1, U$11.P$14, U$12.3IN+
- removed net VDIVRC_D: RC1_4.1, U$11.P$13, U$12.4IN+
- removed net VDIVRC_E: RC2_1.1, U$10.1IN+, U$10.2IN+, U$11.P$12
- removed net VDIVRC_F: RC2_2.1, U$11.P$11
- removed net VDIVRC_G: RC2_3.1, U$10.3IN+, U$11.P$10
- removed net VDIVRC_H: RC2_4.1, U$10.4IN+, U$11.P$9
- new net EN_A: Q2.G
- new net N$25: Q1.D, R1200.CE, R40.2
- new net N$26: Q1.G, Q2.D, R41.2
- net GND: now also ARRAY2.P$10, ARRAY2.P$11, ARRAY2.P$12, ARRAY2.P$13, ARRAY2.P$14, ARRAY2.P$15, ARRAY2.P$16, ARRAY2.P$9, Q2.S, U$11.C1_1, U$11.C2_1, U$11.C3_1, U$11.C4_1, U$13.C1_1, U$13.C2_1, U$13.C3_1, U$13.C4_1; no longer RC1_1.2, RC1_2.2, RC1_3.2, RC1_4.2, RC2_1.2, RC2_2.2, RC2_3.2, RC2_4.2, U$1.P$10, U$1.P$11, U$1.P$12, U$1.P$13, U$1.P$14, U$1.P$15, U$1.P$16, U$1.P$9
- net VDD_A: now also Q1.S, R41.1; no longer R1200.CE
- net VDIV_A: now also ARRAY2.P$1, U$11.C1_2, U$12.1IN+; no longer U$1.P$1, U$11.P$1
- net VDIV_B: now also ARRAY2.P$2, U$11.C2_2, U$12.2IN+; no longer U$1.P$2, U$11.P$2
- net VDIV_C: now also ARRAY2.P$3, U$11.C3_2, U$12.3IN+; no longer U$1.P$3, U$11.P$3
- net VDIV_D: now also ARRAY2.P$4, U$11.C4_2, U$12.4IN+; no longer U$1.P$4, U$11.P$4
- net VDIV_E: now also ARRAY2.P$5, U$10.1IN+, U$13.C1_2; no longer U$1.P$5, U$11.P$5
- net VDIV_F: now also ARRAY2.P$6, U$10.2IN+, U$13.C2_2; no longer U$1.P$6, U$11.P$6
- net VDIV_G: now also ARRAY2.P$7, U$10.3IN+, U$13.C3_2, U$13.C4_2; no longer U$1.P$7, U$11.P$7
- net VDIV_H: now also ARRAY2.P$8, U$10.4IN+; no longer U$1.P$8, U$11.P$8
- net VIN_A: now also R40.1
Other:
- note added: "(adjustable)"
- note removed: "RC Filter"
- moved on the sheet: C1, C10, C11, C12, C13, C14, C15, C16, C17, C18, C19, C2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
