File: modular_battery/battery_module.sch (EAGLE design)
At the start: 138 parts, among them Q1 MOSFET-PCHANNELSOT223, Q2 MOSFET-NCHANNELSMD

Commit message: Board layout
Updated schematic and layed out most of board. Still need to add 30 pin connector.
Parts:
- removed C1, C2, C36, C38: 1uF, SparkFun-Capacitors:CAP0603-CAP
- removed C3, C37: 22pF, SparkFun-Capacitors:CAP0603-CAP
- removed C39, C4: 4.7uF, SparkFun-Passives:CAP0603-CAP
- removed C40, C5: 10nF, SparkFun-Passives:CAP0603-CAP
- removed D1, D8: (no value), SparkFun-DiscreteSemi:DIODESMB
- removed HIGH, HIGH1, HIGH2, HIGH3, HIGH4, HIGH5, HIGH6, HIGH7, LOW, LOW1, LOW2, LOW3, LOW4, LOW5, LOW6, LOW7: IPT004N03L, IPT004N03L:IPT004N03L
- removed L1, L8: (no value), PowerMagnetics (rev18e):WE-LQS_4025_74404043220A
- removed Q1: MOSFET-PCHANNELSOT223, Custom_old:MOSFET-PCHANNELSOT223
- removed Q2: MOSFET-NCHANNELSMD, Custom_old:MOSFET-NCHANNELSMD
- removed R1200: R1200SOT-23-6, Custom_old:R1200SOT-23-6
- removed SI1, SI2, SI3, SI4, SI5, SI6, SI7, SI823: SI8231SOIC16W, Custom_old:SI8231SOIC16W
- removed U$2, U$3, U$4, U$5, U$6, U$7, U$8, U$9: HEADER2, Custom_old:HEADER2
- added C41, C43, C51, C53: 1uF, SparkFun-Capacitors:CAP0603-CAP
- added C42, C52: 22pF, SparkFun-Capacitors:CAP0603-CAP
- added C44, C54: 4.7uF, SparkFun-Passives:CAP0603-CAP
- added C45, C55: (no value), SparkFun-Passives:CAP0603-CAP
- added CN1, CN2, CN3, CN4, CN5, CN6, CN7, CN8, CN9: (no value), adafruit:JST_2PIN-THM
- added D11, D9: (no value), SparkFun-DiscreteSemi:DIODESMB
- added DRIVER11, DRIVER2, DRIVER3, DRIVER4, DRIVER5, DRIVER6, DRIVER7, DRIVER9: SI8231SOIC16W, Custom_old:SI8231SOIC16W
- added L11, L9: (no value), PowerMagnetics (rev18e):WE-LQS_4025_74404043220A
- added NMOS10, NMOS11, NMOS13, NMOS14, NMOS16, NMOS17, NMOS19, NMOS20, NMOS25, NMOS26, NMOS31, NMOS32, NMOS4, NMOS5, NMOS7, NMOS8: IPT004N03L, IPT004N03L:IPT004N03L
- added NMOS12, NMOS15, NMOS18, NMOS21, NMOS27, NMOS33, NMOS6, NMOS9: MOSFET-NCHANNELSMD, Custom_old:MOSFET-NCHANNELSMD
- added PMOS11, PMOS2, PMOS3, PMOS4, PMOS5, PMOS6, PMOS7, PMOS9: MOSFET-PCHANNELSOT223, Custom_old:MOSFET-PCHANNELSOT223
- added R42, R43, R44, R53, R54, R65, R66: 47k, SparkFun-Passives:RESISTOR0603-RES
- added R49, R61: 10k, SparkFun-Resistors:RESISTOR0603
- added R50, R62: 110k, SparkFun-Resistors:RESISTOR0603
- added R51, R63: 2k, SparkFun-Resistors:RESISTOR0603
- added R52, R64: 1k, SparkFun-Resistors:RESISTOR0603
- added VDETECTOR11, VDETECTOR2, VDETECTOR3, VDETECTOR4, VDETECTOR5, VDETECTOR6, VDETECTOR7, VDETECTOR9: BD49XXK__G, Custom_old:BD49XXK__G
- added VREG11, VREG2, VREG3, VREG4, VREG5, VREG6, VREG7, VREG9: R1200SOT-23-6, Custom_old:R1200SOT-23-6
- C10, C15, C20, C25, C30, C35: value 10nF -> (none)
- R1, R30, R35, R5: value 10k -> 47k; device SparkFun-Resistors:RESISTOR0603 -> SparkFun-Passives:RESISTOR0603-RES
- R10: value 10k -> 1k
- R11, R2, R36, R6: value 110k -> 47k; device SparkFun-Resistors:RESISTOR0603 -> SparkFun-Passives:RESISTOR0603-RES
- R12, R17, R3: value 2k -> 47k; device SparkFun-Resistors:RESISTOR0603 -> SparkFun-Passives:RESISTOR0603-RES
- R13: value R1200SOT-23-6 -> 10k; device Custom_old:R1200SOT-23-6 -> SparkFun-Resistors:RESISTOR0603
- R14: value 47k -> 110k
- R15: value 10k -> 2k
- R16: value 110k -> 1k
- R18, R23: value R1200SOT-23-6 -> 47k; device Custom_old:R1200SOT-23-6 -> SparkFun-Passives:RESISTOR0603-RES
- R19: value 47k -> 10k
- R20: value 10k -> 110k
- R21: value 110k -> 2k
- R22: value 2k -> 1k
- R24, R29, R4: device SparkFun-Resistors:RESISTOR0603 -> SparkFun-Passives:RESISTOR0603-RES
- R28: value R1200SOT-23-6 -> 1k; device Custom_old:R1200SOT-23-6 -> SparkFun-Resistors:RESISTOR0603
- R31: value 110k -> 10k
- R32: value 2k -> 110k
- R33: value R1200SOT-23-6 -> 2k; device Custom_old:R1200SOT-23-6 -> SparkFun-Resistors:RESISTOR0603
- R34: value 47k -> 1k
- R37, R7: value 2k -> 10k
- R38, R8: value R1200SOT-23-6 -> 110k; device Custom_old:R1200SOT-23-6 -> SparkFun-Resistors:RESISTOR0603
- R39, R9: value 47k -> 2k
- R40: value 47k -> 1k; device SparkFun-Passives:RESISTOR0603-RES -> SparkFun-Resistors:RESISTOR0603
Connections:
- removed net N$1: L1.1, R1200.LX
- removed net N$26: Q1.G, Q2.D, R41.2
- removed net N$3: R1.1, R1200.VFB, R2.1, R3.2
- removed net N$5: C3.2, R3.1
- new net ENH1_A: PMOS2.D, R11.2, VDETECTOR2.VDD
- new net ENH1_B: PMOS3.D, R17.2, VDETECTOR3.VDD
- new net ENH1_C: PMOS5.D, R29.2, VDETECTOR5.VDD
- new net ENH1_D: PMOS4.D, R23.2, VDETECTOR4.VDD
- new net ENH1_E: PMOS6.D, R35.2, VDETECTOR6.VDD
- new net ENH1_F: PMOS7.D, R41.2, VDETECTOR7.VDD
- new net ENH1_G: PMOS9.D, R53.2, VDETECTOR9.VDD
- new net ENH1_H: PMOS11.D, R65.2, VDETECTOR11.VDD
- new net ENH_A: VDETECTOR2.RES, VREG2.CE
- new net ENH_B: VDETECTOR3.RES, VREG3.CE
- new net ENH_C: VDETECTOR5.RES, VREG5.CE
- new net ENH_D: VDETECTOR4.RES, VREG4.CE
- new net ENH_E: VDETECTOR6.RES, VREG6.CE
- new net ENH_F: VDETECTOR7.RES, VREG7.CE
- new net ENH_G: VDETECTOR9.RES, VREG9.CE
- new net ENH_H: VDETECTOR11.RES, VREG11.CE
- new net EN_B: NMOS9.G
- new net EN_C: NMOS15.G
- new net EN_D: NMOS12.G
- new net EN_E: NMOS18.G
- new net EN_F: NMOS21.G
- new net EN_G: NMOS27.G
- new net EN_H: NMOS33.G
- new net N$27: C32.2, R39.1
- new net N$28: NMOS21.D, PMOS7.G, R42.2
- new net N$33: R49.1, R50.1, R51.2, VREG9.VFB
- new net N$34: L9.1, VREG9.LX
- new net N$35: C42.2, R51.1
- new net N$36: NMOS27.D, PMOS9.G, R54.2
- new net N$41: R61.1, R62.1, R63.2, VREG11.VFB
- new net N$42: L11.1, VREG11.LX
- new net N$43: C52.2, R63.1
- new net N$44: NMOS33.D, PMOS11.G, R66.2
- net 12V_A: now also C7.1, C8.2, D2.A, DRIVER2.VDDB, R8.2, VREG2.VOUT; no longer C2.2, C3.1, D1.A, R1200.VOUT, R2.2, SI823.VDDB
- net 12V_B: now also C12.1, C13.2, D3.A, DRIVER3.VDDB, R14.2, VREG3.VOUT; no longer C7.1, C8.2, D2.A, R6.2, R8.VOUT, SI1.VDDB
- net 12V_C: now also C22.1, C23.2, D5.A, DRIVER5.VDDB, R26.2, VREG5.VOUT; no longer C12.1, C13.2, D3.A, R11.2, R13.VOUT, SI2.VDDB
- net 12V_D: now also DRIVER4.VDDB, R20.2, VREG4.VOUT; no longer R16.2, R18.VOUT, SI3.VDDB
- net 12V_E: now also C27.1, C28.2, D6.A, DRIVER6.VDDB, R32.2, VREG6.VOUT; no longer C22.1, C23.2, D5.A, R21.2, R23.VOUT, SI4.VDDB
- net 12V_F: now also C32.1, C33.2, D7.A, DRIVER7.VDDB, R38.2, VREG7.VOUT; no longer C27.1, C28.2, D6.A, R26.2, R28.VOUT, SI5.VDDB
- net 12V_G: now also C42.1, C43.2, D9.A, DRIVER9.VDDB, R50.2, VREG9.VOUT; no longer C32.1, C33.2, D7.A, R31.2, R33.VOUT, SI6.VDDB
- net 12V_H: now also C52.1, C53.2, D11.A, DRIVER11.VDDB, R62.2, VREG11.VOUT; no longer C37.1, C38.2, D8.A, R36.2, R38.VOUT, SI7.VDDB
- net DISABLE_A: now also DRIVER2.DISABLE, R1.2; no longer SI823.DISABLE
- net DISABLE_B: now also DRIVER3.DISABLE, R2.2; no longer SI1.DISABLE
- net DISABLE_C: now also DRIVER5.DISABLE, R3.2; no longer SI2.DISABLE
- net DISABLE_D: now also DRIVER4.DISABLE, R4.2; no longer SI3.DISABLE
- net DISABLE_E: now also DRIVER6.DISABLE, R44.2; no longer SI4.DISABLE
- net DISABLE_F: now also DRIVER7.DISABLE, R43.2; no longer SI5.DISABLE
- net DISABLE_G: now also DRIVER9.DISABLE, R6.2; no longer SI6.DISABLE
- net DISABLE_H: now also DRIVER11.DISABLE, R5.2; no longer SI7.DISABLE
- net DT_A: now also C10.1, DRIVER2.DT, R10.1; no longer C5.1, R4.1, SI823.DT
- net DT_B: now also C15.1, DRIVER3.DT, R16.1; no longer C10.1, R9.1, SI1.DT
- net DT_C: now also C25.1, DRIVER5.DT, R28.1; no longer C15.1, R14.1, SI2.DT
- net DT_D: now also DRIVER4.DT, R22.1; no longer R19.1, SI3.DT
- net DT_E: now also C30.1, DRIVER6.DT, R34.1; no longer C25.1, R24.1, SI4.DT
- net DT_F: now also C35.1, DRIVER7.DT, R40.1; no longer C30.1, R29.1, SI5.DT
- net DT_G: now also C45.1, DRIVER9.DT, R52.1; no longer C35.1, R34.1, SI6.DT
- net DT_H: now also C55.1, DRIVER11.DT, R64.1; no longer C40.1, R39.1, SI7.DT
- net EN_A: now also NMOS6.G; no longer Q2.G
- net GND: now also C45.2, C55.2, DRIVER11.GNDI, DRIVER2.GNDI, DRIVER3.GNDI, DRIVER4.GNDI, DRIVER5.GNDI, DRIVER6.GNDI, DRIVER7.GNDI, DRIVER9.GNDI, NMOS12.S, NMOS15.S, NMOS18.S, NMOS21.S, NMOS27.S, NMOS33.S, NMOS6.S, NMOS9.S, R1.1, R10.2, R16.2, R2.1, R22.2, R28.2, R3.1, R4.1, R40.2, R43.1, R44.1, R5.1, R52.2, R6.1, R64.2; no longer C40.2, C5.2, Q2.S, R14.2, R19.2, R24.2, R29.2, R39.2, R4.2, R9.2, SI1.GNDI, SI2.GNDI, SI3.GNDI, SI4.GNDI, SI5.GNDI, SI6.GNDI, SI7.GNDI, SI823.GNDI
- net N$10: now also C12.2; no longer R16.1, R17.2, R18.VFB
- net N$11: now also NMOS9.D, PMOS3.G, R18.2; no longer L4.1, R18.LX
- net N$12: now also R19.1, R20.1, R21.2, VREG4.VFB; no longer C17.2, R17.1
- net N$13: now also L4.1, VREG4.LX; no longer R20.1, R21.1, R22.2, R23.VFB
- net N$14: now also C17.2, R21.1; no longer L5.1, R23.LX
- net N$15: now also NMOS12.D, PMOS4.G, R24.2; no longer C22.2, R22.1
- net N$16: now also VREG5.VFB; no longer R28.VFB
- net N$17: now also L5.1, VREG5.LX; no longer L6.1, R28.LX
- net N$18: now also C22.2; no longer C27.2
- net N$19: now also NMOS15.D, PMOS5.G, R30.2; no longer R30.1, R31.1, R32.2, R33.VFB
- net N$2: now also R7.1, R8.1, R9.2, VREG2.VFB; no longer R5.1, R6.1, R7.2, R8.VFB
- net N$20: now also R31.1, R32.1, R33.2, VREG6.VFB; no longer L7.1, R33.LX
- net N$21: now also L6.1, VREG6.LX; no longer C32.2, R32.1
- net N$22: now also C27.2, R33.1; no longer R35.1, R36.1, R37.2, R38.VFB
- net N$23: now also NMOS18.D, PMOS6.G, R36.2; no longer L8.1, R38.LX
- net N$24: now also R38.1, R39.2, VREG7.VFB; no longer C37.2
- net N$25: now also L7.1, VREG7.LX; no longer Q1.D, R1200.CE, R40.2
- net N$4: now also VREG2.LX; no longer R8.LX
- net N$6: now also R9.1; no longer R7.1
- net N$7: now also NMOS6.D, PMOS2.G; no longer R10.1, R11.1, R13.VFB
- net N$8: now also R13.1, R14.1, R15.2, VREG3.VFB; no longer L3.1, R13.LX
- net N$9: now also L3.1, VREG3.LX; no longer C12.2, R12.1
- net PWM_A: now also DRIVER2.PWM; no longer SI823.PWM
- net PWM_B: now also DRIVER3.PWM; no longer SI1.PWM
- net PWM_C: now also DRIVER5.PWM; no longer SI2.PWM
- net PWM_D: now also DRIVER4.PWM; no longer SI3.PWM
- net PWM_E: now also DRIVER6.PWM; no longer SI4.PWM
- net PWM_F: now also DRIVER7.PWM; no longer SI5.PWM
- net PWM_G: now also DRIVER9.PWM; no longer SI6.PWM
- net PWM_H: now also DRIVER11.PWM; no longer SI7.PWM
- net VDD_A: now also ARRAY1.P$4, C6.2, CN1.2, L2.2, NMOS5.9, PMOS2.S, R12.1, VREG2.VDD; no longer ARRAY1.P$1, C1.2, HIGH.9, L1.2, Q1.S, R1200.VDD, R41.1, U$3.1
- net VDD_B: now also ARRAY1.P$3, C11.2, CN4.2, L3.2, NMOS8.9, PMOS3.S, R18.1, VREG3.VDD; no longer ARRAY1.P$2, C6.2, HIGH1.9, L2.2, R8.CE, R8.VDD, U$2.1
- net VDD_C: now also ARRAY1.P$2, C21.2, CN5.2, L5.2, NMOS14.9, PMOS5.S, R30.1, VREG5.VDD; no longer ARRAY1.P$3, C11.2, HIGH2.9, L3.2, R13.CE, R13.VDD, U$4.1
- net VDD_D: now also ARRAY1.P$1, CN7.2, NMOS11.9, PMOS4.S, R24.1, VREG4.VDD; no longer ARRAY1.P$4, HIGH3.9, R18.CE, R18.VDD, U$5.1
- net VDD_E: now also ARRAY1.P$8, C26.2, CN2.2, L6.2, NMOS17.9, PMOS6.S, R36.1, VREG6.VDD; no longer ARRAY1.P$5, C21.2, HIGH4.9, L5.2, R23.CE, R23.VDD, U$6.1
- net VDD_F: now also ARRAY1.P$7, C31.2, CN3.2, L7.2, NMOS20.9, PMOS7.S, R42.1, VREG7.VDD; no longer ARRAY1.P$6, C26.2, HIGH5.9, L6.2, R28.CE, R28.VDD, U$7.1
- net VDD_G: now also ARRAY1.P$6, C41.2, CN6.2, L9.2, NMOS26.9, PMOS9.S, R54.1, VREG9.VDD; no longer ARRAY1.P$7, C31.2, HIGH6.9, L7.2, R33.CE, R33.VDD, U$8.1
- net VDD_H: now also ARRAY1.P$5, C51.2, CN8.2, L11.2, NMOS32.9, PMOS11.S, R66.1, VREG11.VDD; no longer ARRAY1.P$8, C36.2, HIGH7.9, L8.2, R38.CE, R38.VDD, U$9.1
- net VDIV_A: now also ARRAY1.P$13, ARRAY2.P$4, U$12.3IN+; no longer ARRAY1.P$16, ARRAY2.P$1, U$12.1IN+
- net VDIV_B: now also ARRAY1.P$14, ARRAY2.P$3, U$11.C3_2; no longer ARRAY1.P$15, ARRAY2.P$2, U$11.C2_2
- net VDIV_C: now also ARRAY1.P$15, ARRAY2.P$2, U$11.C2_2, U$12.4IN+; no longer ARRAY1.P$14, ARRAY2.P$3, U$11.C3_2, U$12.3IN+
- net VDIV_D: now also ARRAY1.P$16, ARRAY2.P$1, U$12.1IN+; no longer ARRAY1.P$13, ARRAY2.P$4, U$12.4IN+
- net VDIV_E: now also ARRAY1.P$9, ARRAY2.P$8, U$10.2IN+, U$13.C4_2; no longer ARRAY1.P$12, ARRAY2.P$5, U$10.1IN+, U$13.C1_2
- net VDIV_F: now also ARRAY1.P$10, ARRAY2.P$7, U$10.3IN+, U$13.C1_2; no longer ARRAY1.P$11, ARRAY2.P$6, U$10.2IN+, U$13.C2_2
- net VDIV_G: now also ARRAY1.P$11, ARRAY2.P$6, U$10.1IN+; no longer ARRAY1.P$10, ARRAY2.P$7, U$10.3IN+, U$13.C4_2
- net VDIV_H: now also ARRAY1.P$12, ARRAY2.P$5, U$13.C2_2; no longer ARRAY1.P$9, ARRAY2.P$8
- net VIN_A: now also C6.1, C8.1, CN1.1, CN9.1, DRIVER2.GNDB, NMOS4.2, NMOS4.3, NMOS4.4, NMOS4.5, NMOS4.6, NMOS4.7, NMOS4.8, R11.1, R7.2, VDETECTOR2.GND, VREG2.GND; no longer C1.1, C2.1, LOW.2, LOW.3, LOW.4, LOW.5, LOW.6, LOW.7, LOW.8, R1.2, R1200.GND, R40.1, SI823.GNDB, U$3.2
- net VLOGIC: now also DRIVER11.VDDI, DRIVER2.VDDI, DRIVER3.VDDI, DRIVER4.VDDI, DRIVER5.VDDI, DRIVER6.VDDI, DRIVER7.VDDI, DRIVER9.VDDI; no longer SI1.VDDI, SI2.VDDI, SI3.VDDI, SI4.VDDI, SI5.VDDI, SI6.VDDI, SI7.VDDI, SI823.VDDI
- net VOUT+12_A: now also C9.1, D2.C, DRIVER2.VDDA; no longer C4.1, D1.C, SI823.VDDA
- net VOUT+12_B: now also C14.1, D3.C, DRIVER3.VDDA; no longer C9.1, D2.C, SI1.VDDA
- net VOUT+12_C: now also C24.1, D5.C, DRIVER5.VDDA; no longer C14.1, D3.C, SI2.VDDA
- net VOUT+12_D: now also DRIVER4.VDDA; no longer SI3.VDDA
- net VOUT+12_E: now also C29.1, D6.C, DRIVER6.VDDA; no longer C24.1, D5.C, SI4.VDDA
- net VOUT+12_F: now also C34.1, D7.C, DRIVER7.VDDA; no longer C29.1, D6.C, SI5.VDDA
- net VOUT+12_G: now also C44.1, D9.C, DRIVER9.VDDA; no longer C34.1, D7.C, SI6.VDDA
- net VOUT+12_H: now also C54.1, D11.C, DRIVER11.VDDA; no longer C39.1, D8.C, SI7.VDDA
- net VOUT_A: now also C11.1, C13.1, C9.2, CN4.1, DRIVER2.GNDA, DRIVER3.GNDB, NMOS4.9, NMOS5.2, NMOS5.3, NMOS5.4, NMOS5.5, NMOS5.6, NMOS5.7, NMOS5.8, NMOS7.2, NMOS7.3, NMOS7.4, NMOS7.5, NMOS7.6, NMOS7.7, NMOS7.8, R13.2, R17.1, VDETECTOR3.GND, VREG3.GND; no longer C4.2, C6.1, C8.1, HIGH.2, HIGH.3, HIGH.4, HIGH.5, HIGH.6, HIGH.7, HIGH.8, LOW.9, LOW1.2, LOW1.3, LOW1.4, LOW1.5, LOW1.6, LOW1.7, LOW1.8, R5.2, R8.GND, SI1.GNDB, SI823.GNDA, U$2.2
- net VOUT_B: now also C14.2, C21.1, C23.1, CN5.1, DRIVER3.GNDA, DRIVER5.GNDB, NMOS13.2, NMOS13.3, NMOS13.4, NMOS13.5, NMOS13.6, NMOS13.7, NMOS13.8, NMOS7.9, NMOS8.2, NMOS8.3, NMOS8.4, NMOS8.5, NMOS8.6, NMOS8.7, NMOS8.8, R25.2, R29.1, VDETECTOR5.GND, VREG5.GND; no longer C11.1, C13.1, C9.2, HIGH1.2, HIGH1.3, HIGH1.4, HIGH1.5, HIGH1.6, HIGH1.7, HIGH1.8, LOW1.9, LOW2.2, LOW2.3, LOW2.4, LOW2.5, LOW2.6, LOW2.7, LOW2.8, R10.2, R13.GND, SI1.GNDA, SI2.GNDB, U$4.2
- net VOUT_C: now also C24.2, CN7.1, DRIVER4.GNDB, DRIVER5.GNDA, NMOS10.2, NMOS10.3, NMOS10.4, NMOS10.5, NMOS10.6, NMOS10.7, NMOS10.8, NMOS13.9, NMOS14.2, NMOS14.3, NMOS14.4, NMOS14.5, NMOS14.6, NMOS14.7, NMOS14.8, R19.2, R23.1, VDETECTOR4.GND, VREG4.GND; no longer C14.2, HIGH2.2, HIGH2.3, HIGH2.4, HIGH2.5, HIGH2.6, HIGH2.7, HIGH2.8, LOW2.9, LOW3.2, LOW3.3, LOW3.4, LOW3.5, LOW3.6, LOW3.7, LOW3.8, R15.2, R18.GND, SI2.GNDA, SI3.GNDB, U$5.2
- net VOUT_D: now also C26.1, C28.1, CN2.1, DRIVER4.GNDA, DRIVER6.GNDB, NMOS10.9, NMOS11.2, NMOS11.3, NMOS11.4, NMOS11.5, NMOS11.6, NMOS11.7, NMOS11.8, NMOS16.2, NMOS16.3, NMOS16.4, NMOS16.5, NMOS16.6, NMOS16.7, NMOS16.8, R31.2, R35.1, VDETECTOR6.GND, VREG6.GND; no longer C21.1, C23.1, HIGH3.2, HIGH3.3, HIGH3.4, HIGH3.5, HIGH3.6, HIGH3.7, HIGH3.8, LOW3.9, LOW4.2, LOW4.3, LOW4.4, LOW4.5, LOW4.6, LOW4.7, LOW4.8, R20.2, R23.GND, SI3.GNDA, SI4.GNDB, U$6.2
- net VOUT_E: now also C29.2, C31.1, C33.1, CN3.1, DRIVER6.GNDA, DRIVER7.GNDB, NMOS16.9, NMOS17.2, NMOS17.3, NMOS17.4, NMOS17.5, NMOS17.6, NMOS17.7, NMOS17.8, NMOS19.2, NMOS19.3, NMOS19.4, NMOS19.5, NMOS19.6, NMOS19.7, NMOS19.8, R37.2, R41.1, VDETECTOR7.GND, VREG7.GND; no longer C24.2, C26.1, C28.1, HIGH4.2, HIGH4.3, HIGH4.4, HIGH4.5, HIGH4.6, HIGH4.7, HIGH4.8, LOW4.9, LOW5.2, LOW5.3, LOW5.4, LOW5.5, LOW5.6, LOW5.7, LOW5.8, R25.2, R28.GND, SI4.GNDA, SI5.GNDB, U$7.2
- net VOUT_F: now also C34.2, C41.1, C43.1, CN6.1, DRIVER7.GNDA, DRIVER9.GNDB, NMOS19.9, NMOS20.2, NMOS20.3, NMOS20.4, NMOS20.5, NMOS20.6, NMOS20.7, NMOS20.8, NMOS25.2, NMOS25.3, NMOS25.4, NMOS25.5, NMOS25.6, NMOS25.7, NMOS25.8, R49.2, R53.1, VDETECTOR9.GND, VREG9.GND; no longer C29.2, C31.1, C33.1, HIGH5.2, HIGH5.3, HIGH5.4, HIGH5.5, HIGH5.6, HIGH5.7, HIGH5.8, LOW5.9, LOW6.2, LOW6.3, LOW6.4, LOW6.5, LOW6.6, LOW6.7, LOW6.8, R30.2, R33.GND, SI5.GNDA, SI6.GNDB, U$8.2
- net VOUT_G: now also C44.2, C51.1, C53.1, CN8.1, DRIVER11.GNDB, DRIVER9.GNDA, NMOS25.9, NMOS26.2, NMOS26.3, NMOS26.4, NMOS26.5, NMOS26.6, NMOS26.7, NMOS26.8, NMOS31.2, NMOS31.3, NMOS31.4, NMOS31.5, NMOS31.6, NMOS31.7, NMOS31.8, R61.2, R65.1, VDETECTOR11.GND, VREG11.GND; no longer C34.2, C36.1, C38.1, HIGH6.2, HIGH6.3, HIGH6.4, HIGH6.5, HIGH6.6, HIGH6.7, HIGH6.8, LOW6.9, LOW7.2, LOW7.3, LOW7.4, LOW7.5, LOW7.6, LOW7.7, LOW7.8, R35.2, R38.GND, SI6.GNDA, SI7.GNDB, U$9.2
- net VOUT_H: now also C54.2, CN9.2, DRIVER11.GNDA, NMOS31.9, NMOS32.2, NMOS32.3, NMOS32.4, NMOS32.5, NMOS32.6, NMOS32.7, NMOS32.8; no longer C39.2, HIGH7.2, HIGH7.3, HIGH7.4, HIGH7.5, HIGH7.6, HIGH7.7, HIGH7.8, LOW7.9, SI7.GNDA
- net VSENSE_A: now also U$12.3IN-, U$12.3OUT; no longer U$12.1IN-, U$12.1OUT
- net VSENSE_C: now also U$12.4IN-, U$12.4OUT; no longer U$12.3IN-, U$12.3OUT
- net VSENSE_D: now also U$12.1IN-, U$12.1OUT; no longer U$12.4IN-, U$12.4OUT
- net VSENSE_E: now also U$10.2IN-, U$10.2OUT; no longer U$10.1IN-, U$10.1OUT
- net VSENSE_F: now also U$10.3IN-, U$10.3OUT; no longer U$10.2IN-, U$10.2OUT
- net VSENSE_G: now also U$10.1IN-, U$10.1OUT; no longer U$10.3IN-, U$10.3OUT
- net V_HIGH_A: now also DRIVER2.VOA, NMOS5.1; no longer HIGH.1, SI823.VOA
- net V_HIGH_B: now also DRIVER3.VOA, NMOS8.1; no longer HIGH1.1, SI1.VOA
- net V_HIGH_C: now also DRIVER5.VOA, NMOS14.1; no longer HIGH2.1, SI2.VOA
- net V_HIGH_D: now also DRIVER4.VOA, NMOS11.1; no longer HIGH3.1, SI3.VOA
- net V_HIGH_E: now also DRIVER6.VOA, NMOS17.1; no longer HIGH4.1, SI4.VOA
- net V_HIGH_F: now also DRIVER7.VOA, NMOS20.1; no longer HIGH5.1, SI5.VOA
- net V_HIGH_G: now also DRIVER9.VOA, NMOS26.1; no longer HIGH6.1, SI6.VOA
- net V_HIGH_H: now also DRIVER11.VOA, NMOS32.1; no longer HIGH7.1, SI7.VOA
- net V_LOW_A: now also DRIVER2.VOB, NMOS4.1; no longer LOW.1, SI823.VOB
- net V_LOW_B: now also DRIVER3.VOB, NMOS7.1; no longer LOW1.1, SI1.VOB
- net V_LOW_C: now also DRIVER5.VOB, NMOS13.1; no longer LOW2.1, SI2.VOB
- net V_LOW_D: now also DRIVER4.VOB, NMOS10.1; no longer LOW3.1, SI3.VOB
- net V_LOW_E: now also DRIVER6.VOB, NMOS16.1; no longer LOW4.1, SI4.VOB
- net V_LOW_F: now also DRIVER7.VOB, NMOS19.1; no longer LOW5.1, SI5.VOB
- net V_LOW_G: now also DRIVER9.VOB, NMOS25.1; no longer LOW6.1, SI6.VOB
- net V_LOW_H: now also DRIVER11.VOB, NMOS31.1; no longer LOW7.1, SI7.VOB
Other:
- note added: "UVLO"
- note removed: "(adjustable)"
- moved on the sheet: C10, C11, C12, C13, C14, C15, C16, C17, C18, C19, C20, C21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

Commit message: final board layout?
Parts:
- added U$1: 30_HEADER, Custom_old:30_HEADER
Connections:
- new net N$60: U$1.P$28
- new net N$61: U$1.P$26
- new net N$62: U$1.P$30
- new net VENSE_G: U$1.P$4
- net EN_A: now also U$1.P$6
- net EN_B: now also U$1.P$8
- net EN_C: now also U$1.P$10
- net EN_D: now also U$1.P$12
- net EN_E: now also U$1.P$14
- net EN_F: now also U$1.P$16
- net EN_G: now also U$1.P$18
- net EN_H: now also U$1.P$20
- net GND: now also U$1.P$2
- net PWM_A: now also U$1.P$3
- net PWM_B: now also U$1.P$5
- net PWM_C: now also U$1.P$7
- net PWM_D: now also U$1.P$9
- net PWM_E: now also U$1.P$11
- net PWM_F: now also U$1.P$13
- net PWM_G: now also U$1.P$15
- net PWM_H: now also U$1.P$17
- net VLOGIC: now also U$1.P$1
- net VSENSE_A: now also U$1.P$19
- net VSENSE_B: now also U$1.P$21
- net VSENSE_C: now also U$1.P$23
- net VSENSE_D: now also U$1.P$25
- net VSENSE_E: now also U$1.P$27
- net VSENSE_F: now also U$1.P$29
- net VSENSE_G: now also U$1.P$22
- net VSENSE_H: now also U$1.P$24

Commit message: cleanup and CAM
Parts:
- added U$2: FUSE, Custom_old:FUSE
- added VOUT+, VOUT-, VOUT_FUSED: PAD, Custom_old:PAD
Connections:
- new net VOUT_FUSED: U$2.2, VOUT_FUSED.PAD
- net VIN_A: now also VOUT-.PAD
- net VOUT_H: now also U$2.1, VOUT+.PAD
Other:
- moved on the sheet: CN9
Changed lines of the file:
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@@
 <?xml version="1.0" encoding="utf-8"?>
 <!DOCTYPE eagle SYSTEM "eagle.dtd">
-<eagle version="9.2.0">
+<eagle version="9.1.1">
 <drawing>
 <settings>
@@
 <part name="R44" library="SparkFun-Passives" deviceset="RESISTOR" device="0603-RES" value="47k"/>
 <part name="U$1" library="Custom_old" deviceset="30_HEADER" device=""/>
+<part name="VOUT+" library="Custom_old" deviceset="PAD" device=""/>
+<part name="VOUT-" library="Custom_old" deviceset="PAD" device=""/>
+<part name="U$2" library="Custom_old" deviceset="FUSE" device=""/>
+<part name="VOUT_FUSED" library="Custom_old" deviceset="PAD" device=""/>
 </parts>
 <sheets>
@@
 <attribute name="VALUE" x="450.85" y="-99.06" size="1.778" layer="96" rot="R180"/>
 </instance>
-<instance part="CN9" gate="G$1" x="246.38" y="132.08" rot="R180">
-<attribute name="NAME" x="252.73" y="126.365" size="1.778" layer="95" rot="R180"/>
-<attribute name="VALUE" x="252.73" y="137.16" size="1.778" layer="96" rot="R180"/>
+<instance part="CN9" gate="G$1" x="264.16" y="134.62" rot="R180">
+<attribute name="NAME" x="270.51" y="128.905" size="1.778" layer="95" rot="R180"/>
+<attribute name="VALUE" x="270.51" y="139.7" size="1.778" layer="96" rot="R180"/>
 </instance>
 <instance part="R1" gate="G$1" x="-5.08" y="45.72" rot="R90">
@@
 </instance>
 <instance part="U$1" gate="G$1" x="340.36" y="162.56"/>
+<instance part="VOUT+" gate="G$1" x="261.62" y="134.62" rot="R180"/>
+<instance part="VOUT-" gate="G$1" x="261.62" y="132.08" rot="R180"/>
+<instance part="U$2" gate="G$1" x="274.32" y="142.24" rot="R90"/>
+<instance part="VOUT_FUSED" gate="G$1" x="264.16" y="149.86" rot="R180"/>
 </instances>
 <busses>
@@
 <segment>
 <pinref part="CN9" gate="G$1" pin="1"/>
-<wire x1="248.92" y1="129.54" x2="259.08" y2="129.54" width="0.1524" layer="91"/>
-<label x="259.08" y="129.54" size="1.778" layer="95"/>
+<wire x1="266.7" y1="132.08" x2="269.24" y2="132.08" width="0.1524" layer="91"/>
+<label x="276.86" y="132.08" size="1.778" layer="95" xref="yes"/>
+<pinref part="VOUT-" gate="G$1" pin="PAD"/>
+<wire x1="269.24" y1="132.08" x2="276.86" y2="132.08" width="0.1524" layer="91"/>
+<junction x="269.24" y="132.08"/>
 </segment>
 </net>
@@
 <segment>
 <pinref part="CN9" gate="G$1" pin="2"/>
-<wire x1="248.92" y1="132.08" x2="259.08" y2="132.08" width="0.1524" layer="91"/>
-<label x="259.08" y="132.08" size="1.778" layer="95"/>
+<wire x1="266.7" y1="134.62" x2="269.24" y2="134.62" width="0.1524" layer="91"/>
+<label x="276.86" y="134.62" size="1.778" layer="95" xref="yes"/>
+<pinref part="VOUT+" gate="G$1" pin="PAD"/>
+<wire x1="269.24" y1="134.62" x2="274.32" y2="134.62" width="0.1524" layer="91"/>
+<junction x="269.24" y="134.62"/>
+<pinref part="U$2" gate="G$1" pin="1"/>
+<wire x1="274.32" y1="134.62" x2="276.86" y2="134.62" width="0.1524" layer="91"/>
+<junction x="274.32" y="134.62"/>
 </segment>
 </net>
@@
 </segment>
 </net>
+<net name="VOUT_FUSED" class="0">
+<segment>
+<pinref part="U$2" gate="G$1" pin="2"/>
+<pinref part="VOUT_FUSED" gate="G$1" pin="PAD"/>
+<wire x1="271.78" y1="149.86" x2="274.32" y2="149.86" width="0.1524" layer="91"/>
+<label x="274.32" y="149.86" size="1.778" layer="95" xref="yes"/>
+</segment>
+</net>
