File: modular_battery/battery_module.brd (EAGLE design)
At the start: 255.2 x 172.4 mm, 183 parts

Commit message: final board layout?
Parts:
- added U$1: 30_HEADER, Custom_old:2X15_SHROUDED
Connections:
- new net N$60: U$1.28
- new net N$61: U$1.26
- new net N$62: U$1.30
- new net VENSE_G: U$1.4
- net EN_A: now also U$1.6
- net EN_B: now also U$1.8
- net EN_C: now also U$1.10
- net EN_D: now also U$1.12
- net EN_E: now also U$1.14
- net EN_F: now also U$1.16
- net EN_G: now also U$1.18
- net EN_H: now also U$1.20
- net GND: now also U$1.2
- net PWM_A: now also U$1.3
- net PWM_B: now also U$1.5
- net PWM_C: now also U$1.7
- net PWM_D: now also U$1.9
- net PWM_E: now also U$1.11
- net PWM_F: now also U$1.13
- net PWM_G: now also U$1.15
- net PWM_H: now also U$1.17
- net VLOGIC: now also U$1.1
- net VSENSE_A: now also U$1.19
- net VSENSE_B: now also U$1.21
- net VSENSE_C: now also U$1.23
- net VSENSE_D: now also U$1.25
- net VSENSE_E: now also U$1.27
- net VSENSE_F: now also U$1.29
- net VSENSE_G: now also U$1.22
- net VSENSE_H: now also U$1.24
Routing:
- net VSENSE_B: track 1.27 -> 433.4 mm, vias 0 -> 2
- net VSENSE_D: track 1.27 -> 402.6 mm, vias 0 -> 2
- net VSENSE_A: track 1.27 -> 399.8 mm, vias 0 -> 2
- net VSENSE_C: track 1.27 -> 395.9 mm, vias 0 -> 2
- net VSENSE_H: track 1.27 -> 365.6 mm, vias 0 -> 4
- net VSENSE_G: track 1.27 -> 358.2 mm, vias 0 -> 4
- net VSENSE_E: track 1.27 -> 348.0 mm, vias 0 -> 2
- net VSENSE_F: track 1.27 -> 346.8 mm, vias 0 -> 2
- net EN_D: track 0.00 -> 298.2 mm, vias 0 -> 2
- net EN_E: track 0.00 -> 286.3 mm, vias 0 -> 4
- net PWM_D: track 0.00 -> 234.1 mm, vias 0 -> 2
- net EN_F: track 0.00 -> 231.5 mm, vias 0 -> 4
- net PWM_E: track 0.00 -> 226.1 mm, vias 0 -> 8
- net EN_C: track 0.00 -> 184.1 mm, vias 0 -> 8
- net PWM_C: track 0.00 -> 178.7 mm
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- added copper zone on layer 16, net GND
Other:
- board size 255.2 x 172.4 mm -> 308.6 x 172.4 mm

Commit message: cleanup and CAM
Parts:
- added U$2: FUSE, Custom_old:AUTO_FUSE
- added U$3: (no value), Custom_old:DEV
- added VOUT+, VOUT-, VOUT_FUSED: PAD, Custom_old:PAD
- moved U$1 78.7 mm to (5.84, 83.1)
- moved D5 63.6 mm to (164.6, 97.0)
- moved NMOS13 63.6 mm to (146.8, 97.0)
- moved R26 63.6 mm to (164.6, 103.4)
- moved R38 63.6 mm to (164.6, 41.1)
- moved D7 63.6 mm to (164.6, 34.8)
- moved NMOS14 63.6 mm to (146.8, 81.8)
- moved NMOS19 63.6 mm to (146.8, 34.8)
- moved NMOS20 63.6 mm to (146.8, 19.6)
- moved ARRAY1 63.6 mm to (233.2, 67.8)
- moved C10 63.6 mm to (51.6, 121.2)
- moved C12 63.6 mm to (106.2, 103.4)
- moved C15 63.6 mm to (102.4, 121.2)
- moved C16 63.6 mm to (207.8, 80.5)
- moved C17 63.6 mm to (207.8, 103.4)
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Connections:
- new net VOUT_FUSED: U$2.2A, U$2.2B, VOUT_FUSED.PAD
- net VIN_A: now also VOUT-.PAD
- net VOUT_H: now also U$2.1A, U$2.1B, VOUT+.PAD
Routing:
- net EN_G: track 168.6 -> 189.3 mm, vias 4 -> 2
- net EN_D: track 298.2 -> 281.8 mm
- net PWM_D: track 234.1 -> 220.2 mm, vias 2 -> 3
- net PWM_C: track 178.7 -> 164.7 mm
- net PWM_B: track 126.8 -> 112.9 mm
- net PWM_A: track 77.0 -> 63.0 mm
- net VLOGIC: track 531.5 -> 517.6 mm
- net EN_H: track 116.2 -> 128.4 mm
- net VSENSE_C: track 395.9 -> 406.3 mm, vias 2 -> 4
- net VOUT_FUSED: track 0.00 -> 10.1 mm, vias 0 -> 11
- net VSENSE_D: track 402.6 -> 412.3 mm, vias 2 -> 4
- net VSENSE_E: track 348.0 -> 354.1 mm, vias 2 -> 4
- net VSENSE_B: track 433.4 -> 438.6 mm
- net VSENSE_F: track 346.8 -> 351.6 mm, vias 2 -> 3
- net VSENSE_H: track 365.6 -> 370.3 mm, vias 4 -> 5
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- added copper zone on layer 1, net VDD_A
- added copper zone on layer 1, net VDD_B
- added copper zone on layer 1, net VDD_C
- added copper zone on layer 1, net VDD_D
- added copper zone on layer 1, net VDD_E
- added copper zone on layer 1, net VDD_F
- added copper zone on layer 1, net VDD_G
- added copper zone on layer 1, net VDD_H
- added copper zone on layer 1, net VOUT_FUSED
- added copper zone on layer 16, net VOUT_FUSED
- added copper zone on layer 16, net VOUT_H
Other:
- board size 308.6 x 172.4 mm -> 255.3 x 125.9 mm
- board text added: "FUSE"
- board text added: "Modular Battery v1.0 Designed by Jack Proudfoot for Duke Electric Vehicles Feb 24, 2019"
- board text added: "VOUT+"
- board text added: "VOUT-"
