File: H2_v4/main.sch (EAGLE design)
At the start: 15 parts, among them Q1 MOSFET-NCHANNEL, Q2 MOSFET-NCHANNEL, Q3 SOT-23, Q4 SOT-23, Q5 SOT-23, Q6 SOT-23

Commit message: Daily updates. Schematic done, board mostly done
Parts:
- removed Q1, Q2: MOSFET-NCHANNEL, Custom_old (1):MOSFET-NCHANNEL
- added C1, C11, C2, C3, C5: 0.1uF, SparkFun-Passives:CAP0603-CAP
- added C10, C12, C4, C6, C7, C8, C9: 10uF, SparkFun-Passives:CAP1206
- added D3: (no value), SparkFun-DiscreteSemi:DIODESOD123
- added IC1: (no value), 2018:V_REG_78XXV78W
- added LED1, LED2: (no value), SparkFun-LED:LED1206
- added Q7, Q8: MOSFET-NCHANNELDFN5X6, 2018:MOSFET-NCHANNELDFN5X6
- added R1, R16, R17, R2: 1k, SparkFun-Passives:RESISTOR0603-RES
- added R10, R11, R12, R13, R14, R9: 4.7k, SparkFun-Passives:RESISTOR0603-RES
- added R15, R7: 10k, SparkFun-Passives:RESISTOR0603-RES
- added R3, R6: open, SparkFun-Passives:RESISTOR0603-RES
- added R4: 200m, SparkFun-Passives:RESISTOR0603-RES
- added R5: 0, SparkFun-Passives:RESISTOR0603-RES
- added R8: 1.2k, SparkFun-Passives:RESISTOR0603-RES
- added U$10, U$11: PAD, Custom_old (1):PAD
- added U$12: (no value), 2018:CAP-AL_ELECTROLYTIC
- added U$13: HEADER2, Custom_old:HEADER2
- added U$14, U$15, U$18, U$19: SCREW, Custom_old:SCREW
- added U$16, U$17: (no value), 2018:TVS_BIDO-214AB
- added U$20, U$9: HEADER4VALULOK, Custom_old:HEADER4VALULOK
- added U$8: TEENSY_3.0_BASIC, Teensy3.0:TEENSY_3.0_BASIC
- U$1: value PRO-MINI-2 -> SHUNT_KELVIN; device Arduino-clone:PRO-MINI-2 -> 2018:SHUNT_KELVIN
- U$5: value PAD -> HEADER8; device Custom_old (1):PAD -> Custom_old:HEADER8
- U$6: value PAD -> LTC7001; device Custom_old (1):PAD -> 2018:LTC7001
Connections:
- removed net 12V: D1.C, D2.C, U$5.PAD, U$7.POS
- removed net BUZZER: Q5.G
- removed net N$4: Q6.D
- removed net PASS_GATE: Q2.G
- removed net SC_GATE: Q1.G
- new net 5V: C3.2, C8.1, C9.1, IC1.OUT, R5.2, U$6.VCC, U$8.VIN
- new net ACC: C10.1, C4.1, D1.C, D2.C, R6.2, U$20.1, U$5.6, U$5.8, U$7.POS
- new net BUTTON: R15.1, U$13.2, U$8.16/A2
- new net BUZZ_G: Q5.G, U$8.9
- new net CAP_OUT: C5.2, Q8.S, U$10.PAD, U$12.V+, U$17.2, U$6.TS
- new net FAN_H: D3.C, R3.1, R5.1, R6.1, U$5.4
- new net FAN_L: D3.A, Q6.D, U$5.3
- new net FAN_SENSE: C2.1, R7.2, U$8.14/A0
- new net FC_POS: C6.1, C7.1, IC1.IN, Q7.D, Q8.D, R3.2, U$1.I+
- new net FC_RAW: C12.1, U$1.I-, U$16.2, U$3.PAD
- new net LED1: R16.1, U$8.10
- new net LED2: R17.1, U$8.11
- new net N$10: R10.2, U$9.2
- new net N$11: LED2.A, R17.2
- new net N$7: R1.1, U$1.V-
- new net N$8: R2.1, U$1.V+
- new net N$9: Q6.S, R4.2, R7.1
- new net PASS_CTRL: U$6.INP, U$8.7
- new net PASS_G: Q8.G, U$6.TGDN, U$6.TGUP
- new net RX_FLOW: R10.1, R9.1, U$8.0
- new net SCL_EXT: R12.2, U$20.4, U$8.22/A8
- new net SC_G: Q7.G, U$8.8
- new net SDA_EXT: R11.2, U$20.3, U$8.23/A9
- new net THERM: R8.2, U$5.2, U$8.15/A1
- new net TX_FLOW: U$8.1, U$9.3
- net 3.3V: now also C11.1, R11.1, R12.1, R13.1, R14.1, R15.2, R8.1, U$8.3.3V
- net FAN_G: now also U$8.4
- net GND: now also C10.2, C11.2, C12.2, C2.2, C3.1, C4.2, C6.2, C7.2, C8.2, C9.2, IC1.GND, LED1.C, LED2.C, Q7.S, R4.1, R9.2, U$11.PAD, U$12.V-, U$13.1, U$16.1, U$17.1, U$20.2, U$4.PAD, U$5.1, U$6.GND, U$6.OVLO, U$6.VCCUV, U$8.AGND, U$8.GND, U$9.1; no longer Q6.S, U$6.PAD
- net N$1: now also C5.1, U$6.BST; no longer Q1.D, Q2.D, U$3.PAD
- net N$2: now also LED1.A, R16.2; no longer Q1.S, U$4.PAD
- net PRG-: now also U$5.5
- net PRG_G: now also U$8.6
- net SCL: now also R13.2, U$8.19/A5
- net SDA: now also R14.2, U$8.18/A4
- net SHUNT+: now also C1.1, R1.2
- net SHUNT-: now also C1.2, R2.2
- net SV-: now also U$5.7
- net SV_G: now also U$8.5
Other:
- note added: "Fan"
- note added: "High power"
- note removed: "shunt"
- moved on the sheet: D1, D2, Q3, Q4, Q5, Q6

Commit message: First rev of h2v4 finished
Connections:
- net CAP_OUT: now also C6.1, C7.1, IC1.IN, R3.2
- net FAN_SENSE: now also U$8.17/A3; no longer U$8.14/A0
- net FC_POS: no longer C6.1, C7.1, IC1.IN, R3.2
- net PASS_CTRL: now also U$8.3; no longer U$8.7
- net THERM: now also U$8.21/A7; no longer U$8.15/A1
Other:
- note added: "Accessory Battery"
- note added: "Connectors"
- note removed: "ACCESSORY BATTERY"
- moved on the sheet: R10, R15, R8, R9, U$20, U$9

Commit message: fixed pass mosfet
Connections:
- net CAP_OUT: now also Q8.D; no longer C5.2, Q8.S, U$6.TS
- net FC_POS: now also C5.2, Q8.S, U$6.TS; no longer Q8.D
Changed lines of the file:
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@@
 <?xml version="1.0" encoding="utf-8"?>
 <!DOCTYPE eagle SYSTEM "eagle.dtd">
-<eagle version="8.7.1">
+<eagle version="9.1.1">
 <drawing>
 <settings>
@@
 <instance part="U$17" gate="G$1" x="129.54" y="149.86"/>
 <instance part="Q7" gate="G$1" x="91.44" y="147.32"/>
-<instance part="Q8" gate="G$1" x="111.76" y="160.02" rot="R90"/>
+<instance part="Q8" gate="G$1" x="111.76" y="160.02" rot="MR90"/>
 <instance part="U$20" gate="G$1" x="129.54" y="271.78"/>
 <instance part="U$5" gate="G$1" x="170.18" y="274.32"/>
@@
 <segment>
 <wire x1="91.44" y1="160.02" x2="91.44" y2="152.4" width="0.1524" layer="91"/>
-<wire x1="91.44" y1="160.02" x2="106.68" y2="160.02" width="0.1524" layer="91"/>
 <pinref part="U$1" gate="G$1" pin="I+"/>
 <wire x1="73.66" y1="160.02" x2="91.44" y2="160.02" width="0.1524" layer="91"/>
+<label x="83.82" y="160.02" size="1.778" layer="95"/>
+<pinref part="Q7" gate="G$1" pin="D"/>
+<pinref part="Q8" gate="G$1" pin="S"/>
+<wire x1="106.68" y1="160.02" x2="91.44" y2="160.02" width="0.1524" layer="91"/>
 <junction x="91.44" y="160.02"/>
-<label x="83.82" y="160.02" size="1.778" layer="95"/>
-<pinref part="Q8" gate="G$1" pin="D"/>
-<pinref part="Q7" gate="G$1" pin="D"/>
+</segment>
+<segment>
+<pinref part="U$6" gate="G$1" pin="TS"/>
+<label x="304.8" y="73.66" size="1.778" layer="95"/>
+<wire x1="302.26" y1="73.66" x2="327.66" y2="73.66" width="0.1524" layer="91"/>
+<pinref part="C5" gate="G$1" pin="2"/>
+<wire x1="327.66" y1="73.66" x2="327.66" y2="76.2" width="0.1524" layer="91"/>
+<wire x1="327.66" y1="76.2" x2="325.12" y2="76.2" width="0.1524" layer="91"/>
 </segment>
 </net>
@@
 <segment>
 <pinref part="U$10" gate="G$1" pin="PAD"/>
-<wire x1="116.84" y1="160.02" x2="124.46" y2="160.02" width="0.1524" layer="91"/>
 <label x="119.38" y="160.02" size="1.778" layer="95"/>
 <pinref part="U$12" gate="G$1" pin="V+"/>
 <wire x1="124.46" y1="160.02" x2="129.54" y2="160.02" width="0.1524" layer="91"/>
 <wire x1="124.46" y1="154.94" x2="124.46" y2="160.02" width="0.1524" layer="91"/>
-<junction x="124.46" y="160.02"/>
 <pinref part="U$17" gate="G$1" pin="2"/>
 <wire x1="129.54" y1="154.94" x2="129.54" y2="160.02" width="0.1524" layer="91"/>
 <junction x="129.54" y="160.02"/>
-<pinref part="Q8" gate="G$1" pin="S"/>
-</segment>
-<segment>
-<pinref part="U$6" gate="G$1" pin="TS"/>
-<label x="304.8" y="73.66" size="1.778" layer="95"/>
-<wire x1="302.26" y1="73.66" x2="327.66" y2="73.66" width="0.1524" layer="91"/>
-<pinref part="C5" gate="G$1" pin="2"/>
-<wire x1="327.66" y1="73.66" x2="327.66" y2="76.2" width="0.1524" layer="91"/>
-<wire x1="327.66" y1="76.2" x2="325.12" y2="76.2" width="0.1524" layer="91"/>
-</segment>
-<segment>
+<pinref part="Q8" gate="G$1" pin="D"/>
+<wire x1="116.84" y1="160.02" x2="124.46" y2="160.02" width="0.1524" layer="91"/>
+<junction x="124.46" y="160.02"/>
+</segment>
+<segment>
