File: DEV_BMS/main.sch (EAGLE design)
At the start: 75 parts

Commit message: new BMS with CAN and NRF24 radio
Parts:
- removed U$1: INA226, Custom_old:INA226
- removed U$10, U$17, U$19, U$9: HEADER2, Custom_old:HEADER2
- added 12V, CAN1, CAN2, ESTOP1, ESTOP2, I2C_1, I2C_2, TEMP: HEADER2, Custom_old:HEADER2
- added BRAKE: HEADER4VALULOK, Custom_old:HEADER4VALULOK
- added C10, C5: 1uF, SparkFun-Passives:CAP0603-CAP
- added C4: 4.7uF, SparkFun-Passives:CAP0603-CAP
- added IC3: SN65HVD230D, Misaka-IC:SN65HVD230D
- added IC4: INA226, Custom_old:INA226
- added JP1, JP4: JUMPER-SMT_2_NC_TRACE_NO-SILK, SparkFun-Jumpers:JUMPER-SMT_2_NC_TRACE_NO-SILK
- added NRF24: (no value), con-lstb:MA04-2
- added R36: 120, SparkFun-Passives:RESISTOR0603-RES
Connections:
- removed net N$7: IC2.OUT, LED1.A, U$7.COILA
- new net 12V: IC2.OUT, LED1.A, U$18.2, U$7.COILA
- new net BRAKE: BRAKE.1, U$6.21/A7
- new net CANH: CAN1.1, CAN2.1, IC3.CANH, R36.2
- new net CANL: CAN1.2, CAN2.2, IC3.CANL, R36.1
- new net CAN_RX: IC3.RO, U$6.4
- new net CAN_TX: IC3.DI, U$6.3
- new net CE: JP1.2, NRF24.3, U$6.7
- new net CSN: JP4.2, NRF24.4, U$6.8
- new net EN_CAN: IC3.RS, U$6.5
- new net NRF_INT: NRF24.8
- net 3.3: now also IC3.VCC, NRF24.2
- net B_RAW: no longer U$18.1
- net GND: now also 12V.2, BRAKE.2, C10.2, C4.2, C5.2, GPS.3, HALL.2, IC3.GND, IC4.A0, IC4.A1, IC4.GND, NRF24.1, TEMP.1; no longer GPS.2, HALL.3, U$1.A0, U$1.A1, U$1.GND, U$17.1, U$19.1
- net HALL: now also HALL.3; no longer HALL.2
- net IN+: now also IC4.IN+; no longer U$1.IN+
- net IN-: now also IC4.IN-; no longer U$1.IN-
- net LED1: now also JP1.1; no longer U$6.3
- net LED2: now also JP4.1; no longer U$6.21/A7
- net MISO: now also NRF24.7
- net MOSI: now also NRF24.6
- net N$10: now also ESTOP1.2; no longer U$9.2
- net N$12: now also ESTOP1.1, ESTOP2.2; no longer U$10.2, U$9.1
- net N$13: now also ESTOP2.1; no longer U$10.1
- net N$5: now also 12V.1, U$18.1; no longer U$18.2, U$19.2
- net RX1: now also GPS.1; no longer GPS.4
- net SCK: now also NRF24.5
- net SCL: now also I2C_1.2, I2C_2.2, IC4.SCL; no longer U$1.SCL
- net SDA: now also I2C_1.1, I2C_2.1, IC4.SDA; no longer U$1.SDA
- net SD_CS: now also U$6.6; no longer U$6.8
- net THERMISTOR: now also TEMP.2; no longer U$17.2
- net TX1: now also GPS.2; no longer GPS.3
- net VCC: now also BRAKE.4, C10.1, C4.1, C5.1, GPS.4, HALL.4, IC4.VS; no longer GPS.1, HALL.1, U$1.VS
- net V_BAT: now also IC4.VBUS; no longer U$1.VBUS
Other:
- note added: "BATTERY CELL MONITORING"
- note added: "CAN transceiver"
- note added: "CONNECTORS"
- note added: "MCU"
- note added: "NRF24 RADIO"
- note added: "POWER PATH"
- note added: "REGULATORS"
- note added: "SENSORS"
- note added: "on sheet 2"
