File: Joulemeter/main.brd (EAGLE design)
At the start: 88 x 55 mm, 31 parts, among them IC2 SN65HVD230, J1 Boost

Commit message: Joulemeter submit
Parts:
- added J2: (no value), SparkFun-Connectors:1X02
- added U$11, U$12, U$13, U$14: SCREW, Custom_old:M3HOLE
- moved R5 3.64 mm to (33.5, 11.0)
- moved U$7 3.00 mm to (75.0, 12.0)
- moved U$8 3.00 mm to (84.0, 12.0)
- moved U$4 2.07 mm to (84.0, 43.0)
- moved U$3 2.00 mm to (75.0, 43.0)
Connections:
- new net N$4: J2.2, R5.1
- net CANH: now also J2.1; no longer R5.1
Routing:
- net CANL: track 98.6 -> 94.7 mm
- net N$4: track 0.00 -> 3.11 mm
- net CANH: track 83.9 -> 84.7 mm
