File: Joulemeter/main.sch (EAGLE design)
At the start: 31 parts, among them IC2 SN65HVD230, J1 Boost

Commit message: Joulemeter submit
Parts:
- added J2: (no value), SparkFun-Connectors:CONN_02
- added U$11, U$12, U$13, U$14: SCREW, Custom_old:SCREW
Connections:
- new net N$4: J2.2, R5.1
- net CANH: now also J2.1; no longer R5.1
Other:
- moved on the sheet: R5
Changed lines of the file:
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@@
 <part name="C8" library="SparkFun-Capacitors" deviceset="0.1UF" device="-0603-25V-5%" value="0.1uF"/>
 <part name="C9" library="SparkFun-Capacitors" deviceset="10UF" device="-1210-50V-20%" value="10uF"/>
+<part name="J2" library="SparkFun-Connectors" deviceset="CONN_02" device=""/>
+<part name="U$11" library="Custom_old" deviceset="SCREW" device=""/>
+<part name="U$12" library="Custom_old" deviceset="SCREW" device=""/>
+<part name="U$13" library="Custom_old" deviceset="SCREW" device=""/>
+<part name="U$14" library="Custom_old" deviceset="SCREW" device=""/>
 </parts>
 <sheets>
@@
 <attribute name="VALUE" x="137.16" y="83.566" size="1.778" layer="96" align="top-center"/>
 </instance>
-<instance part="R5" gate="G$1" x="190.5" y="99.06" smashed="yes" rot="R270">
-<attribute name="NAME" x="192.024" y="99.06" size="1.778" layer="95" font="vector" rot="R270" align="bottom-center"/>
-<attribute name="VALUE" x="188.976" y="99.06" size="1.778" layer="96" font="vector" rot="R270" align="top-center"/>
+<instance part="R5" gate="G$1" x="200.66" y="99.06" smashed="yes" rot="R270">
+<attribute name="NAME" x="202.184" y="99.06" size="1.778" layer="95" font="vector" rot="R270" align="bottom-center"/>
+<attribute name="VALUE" x="199.136" y="99.06" size="1.778" layer="96" font="vector" rot="R270" align="top-center"/>
 </instance>
 <instance part="C7" gate="G$1" x="119.38" y="91.44" smashed="yes" rot="R180">
@@
 <attribute name="VALUE" x="280.924" y="86.741" size="1.778" layer="96" font="vector"/>
 </instance>
+<instance part="J2" gate="G$1" x="198.12" y="114.3" smashed="yes" rot="R270">
+<attribute name="VALUE" x="193.294" y="116.84" size="1.778" layer="96" font="vector" rot="R270"/>
+<attribute name="NAME" x="203.708" y="116.84" size="1.778" layer="95" font="vector" rot="R270"/>
+</instance>
+<instance part="U$11" gate="G$1" x="264.16" y="60.96" smashed="yes"/>
+<instance part="U$12" gate="G$1" x="264.16" y="55.88" smashed="yes"/>
+<instance part="U$13" gate="G$1" x="264.16" y="50.8" smashed="yes"/>
+<instance part="U$14" gate="G$1" x="264.16" y="45.72" smashed="yes"/>
 </instances>
 <busses>
@@
 <wire x1="180.34" y1="96.52" x2="180.34" y2="93.98" width="0.1524" layer="91"/>
 <pinref part="R5" gate="G$1" pin="2"/>
-<wire x1="180.34" y1="93.98" x2="190.5" y2="93.98" width="0.1524" layer="91"/>
+<wire x1="180.34" y1="93.98" x2="200.66" y2="93.98" width="0.1524" layer="91"/>
 </segment>
 </net>
@@
 <segment>
 <pinref part="IC2" gate="G$1" pin="CANH"/>
-<wire x1="170.18" y1="101.6" x2="180.34" y2="101.6" width="0.1524" layer="91"/>
 <label x="172.72" y="101.6" size="1.778" layer="95"/>
-<pinref part="R5" gate="G$1" pin="1"/>
-<wire x1="180.34" y1="101.6" x2="180.34" y2="104.14" width="0.1524" layer="91"/>
-<wire x1="180.34" y1="104.14" x2="190.5" y2="104.14" width="0.1524" layer="91"/>
+<pinref part="J2" gate="G$1" pin="1"/>
+<wire x1="170.18" y1="101.6" x2="198.12" y2="101.6" width="0.1524" layer="91"/>
+<wire x1="198.12" y1="101.6" x2="198.12" y2="106.68" width="0.1524" layer="91"/>
 </segment>
 </net>
@@
 </segment>
 </net>
+<net name="N$4" class="0">
+<segment>
+<pinref part="R5" gate="G$1" pin="1"/>
+<pinref part="J2" gate="G$1" pin="2"/>
+<wire x1="200.66" y1="104.14" x2="200.66" y2="106.68" width="0.1524" layer="91"/>
+</segment>
+</net>
