File: Controller2019_Guinness/Controller2019_sensorless.sch (EAGLE design)
At the start: 78 parts, among them IC2 L6387EDIP8, IC3 L6387EDIP8, IC4 L6387EDIP8, IC6 MCP2562-E/P, IC7 INA226, J3 FUSE, Q1 MOSFET-NCHANNELPG-HSOF-8-1, Q2 MOSFET-NCHANNELPG-HSOF-8-1, Q3 MOSFET-NCHANNELPG-HSOF-8-1, Q4 MOSFET-NCHANNELPG-HSOF-8-1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

Commit message: idk cleanup
Other:
- note added: "LIST OF BODGES: * on Teensy: throttle to A18 * throttle short R8 * pullups on I2C * pullup on INA ALERT * 3.3V for INA (lolz)"
- note added: "Optional Upgrades: * Hall power cut trace and wire to 15 * 3.3V buck - cut VIN trace and replace with 3.3V"
Changed lines of the file:
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@@
 <wire x1="-10.16" y1="10.16" x2="-48.26" y2="10.16" width="0.1524" layer="97"/>
 <text x="-45.72" y="20.32" size="1.778" layer="97">3V Precision Voltage Reference</text>
+<text x="-66.04" y="96.52" size="1.27" layer="91">LIST OF BODGES:
+* on Teensy: throttle to A18
+* throttle short R8
+* pullups on I2C
+* pullup on INA ALERT
+* 3.3V for INA (lolz)</text>
+<text x="-81.28" y="86.36" size="1.27" layer="91">Optional Upgrades:
+* Hall power cut trace and wire to 15
+* 3.3V buck - cut VIN trace and replace with 3.3V</text>
 </plain>
 <instances>
